Commit message: Multi Robot Capabilities

File: robots/descriptions/go2_description/xacro/gazebo.xacro (robot description, xacro)
@@ -1,18 +1,23 @@
 <?xml version="1.0"?>
-<robot>
-    <!-- Pose publisher plugin for ground truth odometry -->
-    <gazebo>
-        <plugin filename="ignition-gazebo-pose-publisher-system" name="ignition::gazebo::systems::PosePublisher">
-            <publish_link_pose>true</publish_link_pose>
-            <publish_nested_model_pose>true</publish_nested_model_pose>
-            <use_pose_vector_msg>true</use_pose_vector_msg>
-            <update_frequency>10.0</update_frequency>
-        </plugin>
-    </gazebo>
-    <!-- Ignition ros2_control plugin -->
-    <gazebo>
-        <plugin filename="gz_ros2_control-system" name="gz_ros2_control::GazeboSimROS2ControlPlugin">
-            <parameters>$(find go2_description)/config/ros_control/ros_control.yaml</parameters>
-        </plugin>
+<robot xmlns:xacro="http://www.ros.org/wiki/xacro">
+<xacro:macro name="gazebo_setup">
+<!-- Pose publisher plugin for ground truth odometry -->
+<gazebo>
+    <plugin filename="ignition-gazebo-pose-publisher-system" name="ignition::gazebo::systems::PosePublisher">
+        <publish_link_pose>true</publish_link_pose>
+        <publish_nested_model_pose>true</publish_nested_model_pose>
+        <use_pose_vector_msg>true</use_pose_vector_msg>
+        <update_frequency>10.0</update_frequency>
+    </plugin>
+</gazebo>
+<!-- Ignition ros2_control plugin -->
+<xacro:arg name="ros_control_file" default="$(find go2_description)/config/ros_control/ros_control.yaml"/>
+<gazebo>
+    <plugin filename="gz_ros2_control-system" name="gz_ros2_control::GazeboSimROS2ControlPlugin">
+        <ros>
+            <namespace>$(arg robot_name)</namespace>
+        </ros>
+        <parameters>$(find go2_description)/config/ros_control/ros_control.yaml</parameters>
+    </plugin>
     </gazebo>
     <!-- IMU sensor -->
@@ -180,3 +185,4 @@
         <kd>1.0</kd>
     </gazebo>
+</xacro:macro>
 </robot>

File: robots/descriptions/go2_description/xacro/robot.xacro (robot description, xacro)
@@ -2,4 +2,5 @@
 <robot name="go2" xmlns:xacro="http://www.ros.org/wiki/xacro">
     <xacro:arg name="DEBUG" default="false"/>
+    <xacro:arg name="robot_name" default=""/>
     <xacro:include filename="$(find go2_description)/xacro/const.xacro"/>
     <xacro:include filename="$(find go2_description)/xacro/materials.xacro"/>
@@ -110,3 +111,4 @@
     <xacro:leg name="rh" mirror="-1" mirror_dae="False"  front_hind="-1" front_hind_dae="False" />
     <xacro:leg name="lh" mirror="1"  mirror_dae="True"   front_hind="-1" front_hind_dae="False" />
+    <xacro:gazebo_setup/>
 </robot>
